Commit message: switched to torque control with inverse dynamics, and some general refactor

File: urdf/ground.urdf (robot description, URDF)
Before this commit: robot ground_skeleton, 2 links, 1 joints
Links:
- link ground_link: geometry collision box size=11.5 11.5 1; visual box size=11.5 0.05005 11.5
Joints:
- joint ground_joint: origin xyz=0 0 -0.025 rpy=0 0 0 -> xyz=0 0 -0.5 rpy=0 0 0

File: urdf/hrp4.urdf (robot description, URDF)
Before this commit: robot hrp4, 55 links, 54 joints
Links:
- link CHEST_P_LINK: geometry visual mesh filename=../meshes/CHEST_P.dae; visual mesh filename=../meshes/CHEST_R.dae
- link L_ANKLE_P_LINK: geometry visual mesh filename=../meshes/L_ANKLE_P.dae
- link L_ANKLE_R_LINK: geometry visual mesh filename=../meshes/L_ANKLE_R.dae
- link L_ELBOW_P_LINK: geometry visual mesh filename=../meshes/ELBOW_P.dae
- link L_F22_LINK: geometry visual mesh filename=../meshes/F2.dae
- link L_F23_LINK: geometry visual mesh filename=../meshes/F3.dae
- link L_F32_LINK: geometry visual mesh filename=../meshes/F2.dae
- link L_F33_LINK: geometry visual mesh filename=../meshes/F3.dae
- link L_F42_LINK: geometry visual mesh filename=../meshes/F2.dae
- link L_F43_LINK: geometry visual mesh filename=../meshes/F3.dae
- link L_F52_LINK: geometry visual mesh filename=../meshes/F2.dae
- link L_F53_LINK: geometry visual mesh filename=../meshes/F3.dae
- link L_HAND_J0_LINK: geometry visual mesh filename=../meshes/L_THUMB.dae
- link L_HAND_J1_LINK: geometry visual mesh filename=../meshes/L_F1.dae
- link L_HIP_P_LINK: geometry visual mesh filename=../meshes/L_HIP_P.dae
- link L_HIP_R_LINK: geometry visual mesh filename=../meshes/CHEST_P.dae
- link L_HIP_Y_LINK: geometry visual mesh filename=../meshes/HIP_Y.dae
- link L_KNEE_P_LINK: geometry visual mesh filename=../meshes/L_KNEE_P.dae
- link L_SHOULDER_P_LINK: geometry visual mesh filename=../meshes/L_SHOULDER_P.dae
- link L_SHOULDER_R_LINK: geometry visual mesh filename=../meshes/L_SHOULDER_R.dae
- link L_SHOULDER_Y_LINK: geometry visual mesh filename=../meshes/SHOULDER_Y.dae
- link L_WRIST_P_LINK: geometry visual mesh filename=../meshes/WRIST_P.dae
- link L_WRIST_Y_LINK: geometry visual mesh filename=../meshes/L_WRIST_Y.dae
- link NECK_P_LINK: geometry visual mesh filename=../meshes/NECK_P.dae
- link NECK_Y_LINK: geometry visual mesh filename=../meshes/NECK_Y.dae
- link R_ANKLE_P_LINK: geometry visual mesh filename=../meshes/L_ANKLE_P.dae
- link R_ANKLE_R_LINK: geometry visual mesh filename=../meshes/R_ANKLE_R.dae
- link R_ELBOW_P_LINK: geometry visual mesh filename=../meshes/ELBOW_P.dae
- link R_F22_LINK: geometry visual mesh filename=../meshes/F2.dae
- link R_F23_LINK: geometry visual mesh filename=../meshes/F3.dae
- link R_F32_LINK: geometry visual mesh filename=../meshes/F2.dae
- link R_F33_LINK: geometry visual mesh filename=../meshes/F3.dae
- link R_F42_LINK: geometry visual mesh filename=../meshes/F2.dae
- link R_F43_LINK: geometry visual mesh filename=../meshes/F3.dae
- link R_F52_LINK: geometry visual mesh filename=../meshes/F2.dae
- link R_F53_LINK: geometry visual mesh filename=../meshes/F3.dae
- link R_HAND_J0_LINK: geometry visual mesh filename=../meshes/R_THUMB.dae
- link R_HAND_J1_LINK: geometry visual mesh filename=../meshes/R_F1.dae
- link R_HIP_P_LINK: geometry visual mesh filename=../meshes/R_HIP_P.dae
- link R_HIP_R_LINK: geometry visual mesh filename=../meshes/CHEST_P.dae
- link R_HIP_Y_LINK: geometry visual mesh filename=../meshes/HIP_Y.dae
- link R_KNEE_P_LINK: geometry visual mesh filename=../meshes/R_KNEE_P.dae
- link R_SHOULDER_P_LINK: geometry visual mesh filename=../meshes/R_SHOULDER_P.dae
- link R_SHOULDER_R_LINK: geometry visual mesh filename=../meshes/R_SHOULDER_R.dae
- link R_SHOULDER_Y_LINK: geometry visual mesh filename=../meshes/SHOULDER_Y.dae
- link R_WRIST_P_LINK: geometry visual mesh filename=../meshes/WRIST_P.dae
- link R_WRIST_Y_LINK: geometry visual mesh filename=../meshes/R_WRIST_Y.dae
- link body: geometry visual mesh filename=../meshes/WAIST_LINK.dae
- link l_ankle: geometry visual mesh filename=../meshes/L_FOOT.dae
- link l_sole: mass 0.001 -> 1.0; geometry collision box size=0.25 0.13 0.05
- link l_wrist: geometry visual mesh filename=../meshes/L_WRIST_R.dae
- link r_ankle: geometry visual mesh filename=../meshes/R_FOOT.dae
- link r_sole: mass 0.001 -> 1.0; geometry collision box size=0.25 0.13 0.05
- link r_wrist: geometry visual mesh filename=../meshes/R_WRIST_R.dae
- link torso: geometry visual mesh filename=../meshes/CHEST_Y.dae

Commit message: fixed a visualization bug with the ground

File: urdf/ground.urdf (robot description, URDF)
Before this commit: robot ground_skeleton, 2 links, 1 joints
Links:
- link ground_link: geometry collision box size=10 10 1; visual box size=10 10 1
